Commit message: fixed contact instability bug and fixed CoM position for body and right hip

File: src/walker_description/urdf/joint_descriptions.xacro (robot description, xacro)
@@ -9,5 +9,5 @@
   <xacro:property name="hip_joint_friction" value="0.2"/>     <!-- Nm -->
   <xacro:property name="hip_joint_max_velocity" value="10"/>  <!-- rad/s -->
-  <xacro:property name="hip_joint_max_effort" value="30"/>    <!-- Nm -->
+  <xacro:property name="hip_joint_max_effort" value="40"/>    <!-- Nm -->
   <xacro:property name="hip_joint_positive_joint_limit" value="1"/>   <!-- rad -->
   <xacro:property name="hip_joint_negative_joint_limit" value="-1"/>  <!-- rad -->
@@ -16,5 +16,5 @@
   <xacro:property name="carriage_joint_friction" value="0.2"/>     <!-- Nm -->
   <xacro:property name="carriage_joint_max_velocity" value="10"/>  <!-- rad/s -->
-  <xacro:property name="carriage_joint_max_effort" value="30"/>    <!-- Nm -->
+  <xacro:property name="carriage_joint_max_effort" value="40"/>    <!-- Nm -->
   <!-- carriage joint is continuous, so no position joint limits -->
   <!-- leg joint -->
@@ -22,5 +22,5 @@
   <xacro:property name="leg_joint_friction" value="0.2"/>     <!-- N -->
   <xacro:property name="leg_joint_max_velocity" value="10"/>  <!-- m/s -->
-  <xacro:property name="leg_joint_max_effort" value="30"/>    <!-- N -->
+  <xacro:property name="leg_joint_max_effort" value="100"/>    <!-- N -->
   <xacro:property name="leg_joint_positive_joint_limit" value="0.2"/>   <!-- m -->
   <xacro:property name="leg_joint_negative_joint_limit" value="-0.15"/>  <!-- m -->

File: src/walker_description/urdf/walker.xacro (robot description, xacro)
@@ -9,4 +9,6 @@
   <!-- Import joint behavior parameters -->
   <xacro:include filename="$(find walker_description)/urdf/joint_descriptions.xacro" />
+  <!-- Import sim behavior parameters -->
+  <xacro:include filename="$(find walker_description)/urdf/sim_parameters.xacro" />
   <!-- Import transmission file-->
   <xacro:include filename="$(find walker_description)/urdf/transmissions.xacro" />
@@ -19,7 +21,21 @@
   <link
     name="body">
-    <inertial>
-      <origin
-        xyz="0.06218 0.17039 0.15539"
+    <surface>
+      <friction>
+        <ode>
+          <mu>"${ode_mu}"</mu>
+        </ode>
+      </friction>
+      <contact>
+        <ode>
+          <max_vel>0</max_vel>
+          <min_depth>"${ode_min_depth}"</min_depth>
+          <kp>"${ode_kp}"</kp>
+        </ode>
+      </contact>
+    </surface>
+    <inertial>
+      <origin
+        xyz="0.06 -0.16 0.18"
         rpy="0 0 0" />
       <mass
@@ -70,4 +86,17 @@
   <link
     name="left_hip">
+    <surface>
+      <friction>
+        <ode>
+          <mu>"${ode_mu}"</mu>
+        </ode>
+      </friction>
+      <contact>
+        <ode>
+          <min_depth>"${ode_min_depth}"</min_depth>
+          <kp>"${ode_kp}"</kp>
+        </ode>
+      </contact>
+    </surface>
     <inertial>
       <origin
@@ -131,4 +160,17 @@
   <link
     name="left_carriage">
+    <surface>
+      <friction>
+        <ode>
+          <mu>"${ode_mu}"</mu>
+        </ode>
+      </friction>
+      <contact>
+        <ode>
+          <min_depth>"${ode_min_depth}"</min_depth>
+          <kp>"${ode_kp}"</kp>
+        </ode>
+      </contact>
+    </surface>
     <inertial>
       <origin
@@ -190,4 +232,17 @@
   <link
     name="left_leg">
+    <surface>
+      <friction>
+        <ode>
+          <mu>"${ode_mu}"</mu>
+        </ode>
+      </friction>
+      <contact>
+        <ode>
+          <min_depth>"${ode_min_depth}"</min_depth>
+          <kp>"${ode_kp}"</kp>
+        </ode>
+      </contact>
+    </surface>
     <inertial>
       <origin
@@ -251,8 +306,24 @@
   <link
     name="right_hip">
-    <inertial>
-      <origin
+    <surface>
+      <friction>
+        <ode>
+          <mu>"${ode_mu}"</mu>
+        </ode>
+      </friction>
+      <contact>
+        <ode>
+          <min_depth>"${ode_min_depth}"</min_depth>
+          <kp>"${ode_kp}"</kp>
+        </ode>
+      </contact>
+    </surface>
+    <inertial>
+      <origin
+        xyz="0.07 0 0.03"
+        rpy="0 0 0" />
+      <!-- <origin
         xyz="0.06218 0.17039 0.15539"
-        rpy="0 0 0" />
+        rpy="0 0 0" /> -->
       <mass
         value="0.36941" />
@@ -312,4 +383,17 @@
   <link
     name="right_carriage">
+    <surface>
+      <friction>
+        <ode>
+          <mu>"${ode_mu}"</mu>
+        </ode>
+      </friction>
+      <contact>
+        <ode>
+          <min_depth>"${ode_min_depth}"</min_depth>
+          <kp>"${ode_kp}"</kp>
+        </ode>
+      </contact>
+    </surface>
     <inertial>
       <origin
@@ -371,4 +455,17 @@
   <link
     name="right_leg">
+    <surface>
+      <friction>
+        <ode>
+          <mu>"${ode_mu}"</mu>
+        </ode>
+      </friction>
+      <contact>
+        <ode>
+          <min_depth>"${ode_min_depth}"</min_depth>
+          <kp>"${ode_kp}"</kp>
+        </ode>
+      </contact>
+    </surface>
     <inertial>
       <origin
